File: Electronic/fcu/fcu-display-driver1.sch (KiCad schematic (older format))
At the start: 8 parts

Commit message: Update fcu schemas and libraries
Parts:
- removed ALT201, ALT202, ALT203, ALT204, ALT205, SPEED201, SPEED202, SPEED203: HDSP-7403, Display_7Segment:HDSP-7401, symbol Display_Character:HDSP-7403
- added ALT1, ALT2, ALT3, ALT4, ALT5, SPEED1, SPEED2, SPEED3: HDSP-7401, Display_7Segment:HDSP-7401, symbol Display_Character:HDSP-7401
Other:
- note added: "Note : segments and digits are inverted because digits are Common Anode (CA)."
