File: Electronic/fcu/fcu-display-driver2.sch (KiCad schematic (older format))
At the start: 8 parts

Commit message: Update fcu schemas and libraries
Parts:
- removed HDG301, HDG302, HDG303, VS301, VS302, VS303, VS304, VS305: HDSP-7403, Display_7Segment:HDSP-7401, symbol Display_Character:HDSP-7403
- added HDG1, HDG2, HDG3, VS1, VS2, VS3, VS4, VS5: HDSP-7401, Display_7Segment:HDSP-7401, symbol Display_Character:HDSP-7401
Other:
- note added: "Note : segments and digits are inverted because digits are Common Anode (CA)."
