File: Electronic/fcu/fcu-display-driver3.sch (KiCad schematic (older format))
At the start: 17 parts

Commit message: Update fcu schemas and libraries
Parts:
- renumbered PadALT401 to PadALT1, PaveFPA401 to PadFPA1, PaveFPA402 to PadFPA2, PaveHDG401 to PadHDG1, PaveHDG402 to PadHDG2, PadLVLCH401 to PadLVLCH1, PadLine401 to PadLine1, PadLine402 to PadLine2, PaveMach401 to PadMach1, PaveSpeed401 to PadSpeed1, PaveTRK401 to PadTRK1, PaveTRK402 to PadTRK2, PaveVS401 to PadVS1, PaveVS402 to PadVS2
Connections:
- wire segments 118 -> 120
- no-connect marks 6 -> 7

Commit message: Update references to symbol in right library
Parts:
- PadALT1, PadFPA1, PadFPA2, PadHDG1, PadHDG2, PadLVLCH1, PadLine1, PadLine2, PadMach1, PadSpeed1, PadTRK1, PadTRK2, PadVS1, PadVS2: symbol fcu-display-rescue:LedPave-home-cockpit-library -> home-cockpit-symbols:LedPave
Connections:
- wire segments 120 -> 91
Changed lines of the file:
@@
 Wire Wire Line
 	7750 2600 7750 2850
-Wire Wire Line
-	7000 2600 7000 2850
-Wire Wire Line
-	7600 2950 7600 3250
-Wire Wire Line
-	6700 2950 6700 3250
-Wire Wire Line
-	5250 2650 5250 2850
-Wire Wire Line
-	5850 2950 5850 3250
-Wire Wire Line
-	4400 2450 4400 2850
-Wire Wire Line
-	5000 2950 5000 3250
-Wire Wire Line
-	7900 1400 7900 1600
-Wire Wire Line
-	8500 1700 8500 2100
-Wire Wire Line
-	7050 1400 7050 1600
-Wire Wire Line
-	7650 1700 7650 2100
-Wire Wire Line
-	6100 1400 6100 1600
-Wire Wire Line
-	6700 1600 6700 1700
-Wire Wire Line
-	5250 1400 5250 1600
-Wire Wire Line
-	5000 1600 5000 1700
-$Comp
-L fcu-display-rescue:LedPave-home-cockpit-library PadLine?
+$Comp
+L home-cockpit-symbols:LedPave PadLine?
 U 1 1 60360EA3
 P 8100 2750
@@
 $EndComp
 $Comp
-L fcu-display-rescue:LedPave-home-cockpit-library PadLine?
+L home-cockpit-symbols:LedPave PadLine?
 U 1 1 60366B4C
 P 7300 2750
@@
 $EndComp
 $Comp
-L fcu-display-rescue:LedPave-home-cockpit-library PadLine?
+L home-cockpit-symbols:LedPave PadLine?
 U 1 1 60366EBA
 P 6400 2750
@@
 $EndComp
 $Comp
-L fcu-display-rescue:LedPave-home-cockpit-library PadLine?
+L home-cockpit-symbols:LedPave PadLine?
 U 1 1 603671F5
 P 5550 2750
@@
 $EndComp
 $Comp
-L fcu-display-rescue:LedPave-home-cockpit-library PaveTRK?
+L home-cockpit-symbols:LedPave PaveTRK?
 U 1 1 603692E6
 P 4700 2750
@@
 $EndComp
 Wire Wire Line
-	4400 2950 4400 2850
-Connection ~ 4400 2850
-Wire Wire Line
-	5000 2850 5000 2950
-Connection ~ 5000 2950
-Wire Wire Line
-	5250 2950 5250 2850
-Connection ~ 5250 2850
-Wire Wire Line
-	5850 2950 5850 2850
-Connection ~ 5850 2950
-Wire Wire Line
-	6100 2650 6100 2850
-Wire Wire Line
-	6100 2950 6100 2850
-Connection ~ 6100 2850
-Wire Wire Line
-	6700 2950 6700 2850
-Connection ~ 6700 2950
-Wire Wire Line
-	7000 2950 7000 2850
-Connection ~ 7000 2850
-Wire Wire Line
-	7600 2850 7600 2950
-Connection ~ 7600 2950
-Wire Wire Line
-	8400 2950 8400 3250
-Wire Wire Line
 	7750 2950 7800 2950
 Wire Wire Line
@@
 Wire Wire Line
 	7750 2850 7750 2950
-Wire Wire Line
-	8400 2850 8400 2950
-Connection ~ 8400 2950
-$Comp
-L fcu-display-rescue:LedPave-home-cockpit-library PaveFPA?
+$Comp
+L home-cockpit-symbols:LedPave PaveFPA?
 U 1 1 603D00CB
 P 8200 1500
@@
 $EndComp
 $Comp
-L fcu-display-rescue:LedPave-home-cockpit-library PaveVS?
+L home-cockpit-symbols:LedPave PaveVS?
 U 1 1 603D1EF3
 P 7350 1500
@@
 $EndComp
 $Comp
-L fcu-display-rescue:LedPave-home-cockpit-library PaveVS?
+L home-cockpit-symbols:LedPave PaveVS?
 U 1 1 603D2274
 P 6400 1500
@@
 $EndComp
 $Comp
-L fcu-display-rescue:LedPave-home-cockpit-library PaveVS?
+L home-cockpit-symbols:LedPave PaveVS?
 U 1 1 603D2560
 P 5550 1500
@@
 $EndComp
 $Comp
-L fcu-display-rescue:LedPave-home-cockpit-library PaveVS?
+L home-cockpit-symbols:LedPave PaveVS?
 U 1 1 603D2F30
 P 4700 1500
@@
 	1    0    0    -1
 $EndComp
-Connection ~ 5000 1700
-Wire Wire Line
-	5000 1700 5000 2100
-Wire Wire Line
-	4400 1700 4400 1600
-Wire Wire Line
-	5250 1700 5250 1600
-Connection ~ 5250 1600
-Connection ~ 6700 1700
-Wire Wire Line
-	6700 1700 6700 2100
-Wire Wire Line
-	6100 1700 6100 1600
-Connection ~ 6100 1600
-Wire Wire Line
-	7650 1600 7650 1700
-Connection ~ 7650 1700
-Wire Wire Line
-	7050 1700 7050 1600
-Connection ~ 7050 1600
-Wire Wire Line
-	8500 1700 8500 1600
-Connection ~ 8500 1700
-Wire Wire Line
-	7900 1700 7900 1600
-Connection ~ 7900 1600
 Wire Wire Line
 	4200 2100 4200 2850
@@
 	1700 2850 4200 2850
 $Comp
-L fcu-display-rescue:LedPave-home-cockpit-library PadALT?
+L home-cockpit-symbols:LedPave PadALT?
 U 1 1 6044F716
 P 6100 4600
@@
 $EndComp
 $Comp
-L fcu-display-rescue:LedPave-home-cockpit-library PadLVLCH?
+L home-cockpit-symbols:LedPave PadLVLCH?
 U 1 1 6044F71C
 P 7300 4600
@@
 $EndComp
 $Comp
-L fcu-display-rescue:LedPave-home-cockpit-library PadLine?
+L home-cockpit-symbols:LedPave PadLine?
 U 1 1 6044F722
 P 9750 4600
@@
 $EndComp
 $Comp
-L fcu-display-rescue:LedPave-home-cockpit-library PadLine?
+L home-cockpit-symbols:LedPave PadLine?
 U 1 1 6044F728
 P 8500 4600
@@
 $EndComp
 Wire Wire Line
-	10050 4700 10050 4800
-Wire Wire Line
 	9400 4700 9450 4700
 Wire Wire Line
@@
 Wire Wire Line
 	9400 4800 9450 4800
-Wire Wire Line
-	8200 4700 8200 4800
-Wire Wire Line
-	8800 4700 8800 4800
 Wire Wire Line
 	6950 4700 7000 4700
@@
 Wire Wire Line
 	7650 4700 7650 4800
-Wire Wire Line
-	6400 4700 6400 4800
-Wire Wire Line
-	5800 4700 5800 4800
 Connection ~ 3950 3850
 Entry Wire Line
@@
 Entry Wire Line
 	5700 3850 5800 3950
-Wire Wire Line
-	8200 3950 8200 4700
-Wire Wire Line
-	5800 3950 5800 4700
-Connection ~ 10050 4800
 Wire Notes Line
 	10300 3750 4300 3750
-Connection ~ 5800 4700
-Connection ~ 8200 4700
 Entry Wire Line
 	6850 3850 6950 3950
@@
 Connection ~ 9400 4700
 Wire Wire Line
-	10050 4800 10050 5200
-Wire Wire Line
 	7650 4800 7650 5200
 Wire Wire Line
 	7650 5200 8800 5200
-Wire Wire Line
-	8800 4800 8800 5200
-Connection ~ 8800 4800
 Connection ~ 8800 5200
 Wire Wire Line
 	8800 5200 10050 5200
-Wire Wire Line
-	6400 4800 6400 5200
-Connection ~ 6400 4800
 Text Label 5800 4100 0    50   ~ 0
 Dr3SegD
@@
 $EndComp
 Wire Wire Line
-	4400 2000 4400 1700
-Connection ~ 4400 1700
-Wire Wire Line
 	7050 1400 7900 1400
-Wire Wire Line
-	7050 2000 7050 1700
-Connection ~ 7050 1700
 $Comp
 L power:PWR_FLAG #FLG?
@@
 	0    1    1    0
 $EndComp
-Wire Wire Line
-	5250 2000 5250 1700
-Connection ~ 5250 1700
 $Comp
 L power:PWR_FLAG #FLG?
@@
 	0    1    1    0
 $EndComp
-Wire Wire Line
-	7000 3200 7000 2950
-Connection ~ 7000 2950
-Wire Wire Line
-	5250 3200 5250 2950
-Connection ~ 5250 2950
-Wire Wire Line
-	4400 3200 4400 2950
-Connection ~ 4400 2950
 $Comp
 L power:PWR_FLAG #FLG?
@@
 Wire Wire Line
 	5000 2100 5850 2100
-Wire Wire Line
-	5850 1600 5850 1700
-Wire Wire Line
-	5850 1700 5850 2100
-Connection ~ 5850 1700
 Connection ~ 5850 2100
 Wire Wire Line
 	5850 2100 6700 2100
+Wire Wire Line
+	7600 2850 7600 3250
+Wire Wire Line
+	6700 2850 6700 3250
+Wire Wire Line
+	5850 2850 5850 3250
+Wire Wire Line
+	5000 2850 5000 3250
+Wire Wire Line
+	7900 1400 7900 1700
+Wire Wire Line
+	8500 1600 8500 2100
+Wire Wire Line
+	7650 1600 7650 2100
+Wire Wire Line
+	6100 1400 6100 1700
+Wire Wire Line
+	6700 1600 6700 2100
+Wire Wire Line
+	5000 1600 5000 2100
+Wire Wire Line
+	6100 2650 6100 2950
+Wire Wire Line
+	8400 2850 8400 3250
+Wire Wire Line
+	4400 1600 4400 2000
+Wire Wire Line
+	10050 4700 10050 5200
+Wire Wire Line
+	8200 3950 8200 4800
+Wire Wire Line
+	8800 4700 8800 5200
+Wire Wire Line
+	6400 4700 6400 5200
+Wire Wire Line
+	5800 3950 5800 4800
+Wire Wire Line
+	7050 1400 7050 2000
+Wire Wire Line
+	5250 1400 5250 2000
+Wire Wire Line
+	7000 2600 7000 3200
+Wire Wire Line
+	5250 2650 5250 3200
+Wire Wire Line
+	4400 2450 4400 3200
+Wire Wire Line
+	5850 1600 5850 2100
 Wire Bus Line
 	3950 3850 3950 4900

Commit message: Update electornic schema of FCU MotherBoard and Display. Replace MAX7219 for leds to dedicated TLC5917.
Parts:
- added PadLAT1: LedPad, home-cockpit-footprints:PadLed-KingBright-DE-2YD, symbol home-cockpit-symbols:LedPad
- PadALT1, PadFPA1, PadFPA2, PadHDG1, PadHDG2, PadLVLCH1, PadLine1, PadLine2, PadMach1, PadSpeed1, PadTRK1, PadTRK2, PadVS1, PadVS2: value LedPave-home-cockpit-library -> LedPad; symbol home-cockpit-symbols:LedPave -> home-cockpit-symbols:LedPad
Connections:
- net labels added: LedManagedALT, LedManagedHDG, LedManagedSpeed, LedPadFPA, LedPadHDG, LedPadLAT, LedPadMACH, LedPadSPD, LedPadStaticALT, LedPadStaticLines, LedPadTRK, LedPadVS, Vcc12V
- net labels removed: Dr3Dig0, Dr3Dig1, Dr3Dig2, Dr3Dig3, Dr3Dig4, Dr3Dig5, Dr3Dig6, Dr3Dig7, Dr3SegA, Dr3SegB, Dr3SegC, Dr3SegD, Dr3SegDP, Dr3SegE, Dr3SegF, Dr3SegG
- wire segments 91 -> 105
- no-connect marks 7 -> 0
Other:
- note removed: "Digit 0"
- note removed: "Digit 1"
