File: Electronic/fcu/fcu-display.sch (KiCad schematic (older format))
At the start: 1 part, among them U101 Connector-FPC-50pins

Commit message: Update fcu schemas and libraries
Connections:
- no-connect marks 3 -> 2

Commit message: Update electornic schema of FCU MotherBoard and Display. Replace MAX7219 for leds to dedicated TLC5917.
Parts:
- removed U101: Connector-FPC-50pins, home-cockpit-footprints:Connector-FPC-50pins-0.5mm, symbol home-cockpit-symbols:Connector-FPC-50pins
- added DisplayConnector1: Connector-FPC-50pins, home-cockpit-footprints:Connector-FPC-50pins-0.5mm, symbol home-cockpit-symbols:Connector-FPC-50pins
Connections:
- net labels added: +12V, LedManagedALT, LedManagedHDG, LedManagedSpeed, LedPadFPA, LedPadHDG, LedPadLAT, LedPadMACH, LedPadSPD, LedPadStaticALT, LedPadStaticLines, LedPadTRK, LedPadVS, Vcc12V
- net labels removed: Dr3Dig0, Dr3Dig1, Dr3Dig2, Dr3Dig3, Dr3Dig4, Dr3Dig5, Dr3Dig6, Dr3Dig7, Dr3SegA, Dr3SegB, Dr3SegC, Dr3SegD, Dr3SegDP, Dr3SegE, Dr3SegF, Dr3SegG
- wire segments 48 -> 54
- no-connect marks 2 -> 5
