File: Electronic/fcu/fcu-mb-display-drivers.sch (KiCad schematic (older format))
At the start: 6 parts, among them U1 MAX7219, U2 MAX7219, U3 MAX7219

Commit message: Finalise first FCU PCB version
Parts:
- renumbered U2 to DriverHdgVs1, U3 to DriverOther1, U1 to DriverSpeedAlt1
Changed lines of the file:
@@
 P 3950 3650
 AR Path="/602F293B" Ref="U?"  Part="1"
-AR Path="/602DB478/602F293B" Ref="U1"  Part="1"
-F 0 "U1" H 3950 4831 50  0000 C CNN
+AR Path="/602DB478/602F293B" Ref="DriverSpeedAlt1"  Part="1"
+F 0 "DriverSpeedAlt1" H 3950 4831 50  0000 C CNN
 F 1 "MAX7219" H 3950 4740 50  0000 C CNN
 F 2 "Package_DIP:DIP-24_W7.62mm_Socket" H 3900 3700 50  0001 C CNN
@@
 P 5750 3650
 AR Path="/602F2941" Ref="U?"  Part="1"
-AR Path="/602DB478/602F2941" Ref="U2"  Part="1"
-F 0 "U2" H 5750 4831 50  0000 C CNN
+AR Path="/602DB478/602F2941" Ref="DriverHdgVs1"  Part="1"
+F 0 "DriverHdgVs1" H 5750 4831 50  0000 C CNN
 F 1 "MAX7219" H 5750 4740 50  0000 C CNN
 F 2 "Package_DIP:DIP-24_W7.62mm_Socket" H 5700 3700 50  0001 C CNN
@@
 P 7400 3650
 AR Path="/602F2947" Ref="U?"  Part="1"
-AR Path="/602DB478/602F2947" Ref="U3"  Part="1"
-F 0 "U3" H 7400 4831 50  0000 C CNN
+AR Path="/602DB478/602F2947" Ref="DriverOther1"  Part="1"
+F 0 "DriverOther1" H 7400 4831 50  0000 C CNN
 F 1 "MAX7219" H 7400 4740 50  0000 C CNN
 F 2 "Package_DIP:DIP-24_W7.62mm_Socket" H 7350 3700 50  0001 C CNN

Commit message: Update electornic schema of FCU MotherBoard and Display. Replace MAX7219 for leds to dedicated TLC5917.
Parts:
- removed DriverOther1: MAX7219, Package_DIP:DIP-24_W7.62mm_Socket, symbol Driver_LED:MAX7219
- added C3, C4: 0,1µF, Capacitor_THT:C_Disc_D7.0mm_W2.5mm_P5.00mm, symbol Device:C
- added C5, C6, C7: 1µF, Capacitor_THT:C_Disc_D7.0mm_W2.5mm_P5.00mm, symbol Device:C_Small
- added DriverLed1, DriverLed2, DriverLed3: TLC5917IN, home-cockpit-footprints:Texas_Instruments-TLC5917IN-Manufacturer_Recommended, symbol home-cockpit-symbols:TLC5917IN
- added R29, R30: 9,53kohms, Resistor_THT:R_Axial_DIN0207_L6.3mm_D2.5mm_P10.16mm_Horizontal, symbol Device:R
Connections:
- net labels added: DriverDigitClock, DriverDigitData, DriverDigitLoad, DriverLedClock, DriverLedData, DriverLedLoad, LedKorryAP1, LedKorryAP2, LedKorryAPPR, LedKorryATHR, LedKorryEXPED, LedKorryLoc, LedManagedALT, LedManagedHDG, LedManagedSpeed, LedOutputEnable, LedPadFPA, LedPadHDG, LedPadLAT, LedPadMACH, LedPadSPD, LedPadStaticALT, LedPadStaticLines, LedPadTRK, LedPadVS
- net labels removed: Dr3Dig0, Dr3Dig1, Dr3Dig2, Dr3Dig3, Dr3Dig4, Dr3Dig5, Dr3Dig6, Dr3Dig7, Dr3SegA, Dr3SegB, Dr3SegC, Dr3SegD, Dr3SegDP, Dr3SegE, Dr3SegF, Dr3SegG, DriverClock, DriverData, DriverLoad
- wire segments 84 -> 124
- no-connect marks 1 -> 8
Other:
- note added: "DriverLed1 :\nLed PAD"
- note added: "DriverLed2 :\nLed KORRY"
- note added: "DriverLed3 :\nLed Managed mode"
- note added: "DriverSegment1 :\nSpeed digits\nAltitude digits"
- note added: "DriverSegment2 :\nHDG digits\nVS digits"
- note removed: "Driver1 :\nSpeed digits\nAltitude digits"
- note removed: "Driver2 :\nHDG digits\nVS digits"
- note removed: "Driver3 :\nDigit 0 : Display Led PAD (on Display PCB)\nDigit 1 : Display Led PAD (on Display PCB)\nDigit 2 : FCU Korry green Led"

Commit message: Adjust resistor values for TLC5917
Parts:
- R29, R3: value 9,53kohms -> 1kohms
- R30: value 9,53kohms -> 2kohms
Other:
- note added: "DriverLed1 :\nLed PAD (20mA)"
- note added: "DriverLed2 :\nLed KORRY (20mA)"
- note added: "DriverLed3 :\nLed Managed mode (10mA)"
- note removed: "DriverLed1 :\nLed PAD"
- note removed: "DriverLed2 :\nLed KORRY"
- note removed: "DriverLed3 :\nLed Managed mode"
Changed lines of the file:
@@
 $EndComp
 Text Notes 9050 1400 0    50   ~ 0
-DriverLed1 :\nLed PAD
+DriverLed1 :\nLed PAD (20mA)
 Text Notes 3800 5250 0    50   ~ 0
 DriverSegment2 :\nHDG digits\nVS digits
@@
 AR Path="/602DB478/6072A07A" Ref="R3"  Part="1"
 F 0 "R3" V 7400 2400 50  0000 C CNN
-F 1 "9,53kohms" V 7600 2600 50  0000 R CNN
+F 1 "1kohms" V 7600 2600 50  0000 R CNN
 F 2 "Resistor_THT:R_Axial_DIN0207_L6.3mm_D2.5mm_P10.16mm_Horizontal" V 7430 2400 50  0001 C CNN
 F 3 "~" H 7500 2400 50  0001 C CNN
@@
 AR Path="/602DB478/608677D2" Ref="R29"  Part="1"
 F 0 "R29" V 7400 4350 50  0000 C CNN
-F 1 "9,53kohms" V 7600 4550 50  0000 R CNN
+F 1 "1kohms" V 7600 4550 50  0000 R CNN
 F 2 "Resistor_THT:R_Axial_DIN0207_L6.3mm_D2.5mm_P10.16mm_Horizontal" V 7430 4350 50  0001 C CNN
 F 3 "~" H 7500 4350 50  0001 C CNN
@@
 	6050 3350 7000 3350
 Text Notes 9050 3350 0    50   ~ 0
-DriverLed2 :\nLed KORRY
+DriverLed2 :\nLed KORRY (20mA)
 Text GLabel 8100 4950 2    50   Input ~ 0
 LedManagedSpeed
@@
 AR Path="/602DB478/60A75A39" Ref="R30"  Part="1"
 F 0 "R30" V 7400 6350 50  0000 C CNN
-F 1 "9,53kohms" V 7600 6550 50  0000 R CNN
+F 1 "2kohms" V 7600 6550 50  0000 R CNN
 F 2 "Resistor_THT:R_Axial_DIN0207_L6.3mm_D2.5mm_P10.16mm_Horizontal" V 7430 6350 50  0001 C CNN
 F 3 "~" H 7500 6350 50  0001 C CNN
@@
 	6050 5350 7000 5350
 Text Notes 9050 5350 0    50   ~ 0
-DriverLed3 :\nLed Managed mode
+DriverLed3 :\nLed Managed mode (10mA)
 Wire Wire Line
 	7000 3450 6050 3450
